Commit message: updated the file paths for meshes to be relative

File: src/isaac_so_arm101/robots/pingti/PingTi_Arm_5DOF_v4_copy.xacro (robot description, xacro)
@@ -13,5 +13,5 @@
     <origin xyz="0 0 0" rpy="0 0 0"/>
     <geometry>
-      <mesh filename="/home/cirp-lab/moore/prefab_robots/PingTi_Arm_v3/PingTi_Arm_5DOF_v4_copy_description/meshes/base_link.stl" scale="0.001 0.001 0.001"/>
+      <mesh filename="meshes/base_link.stl" scale="0.001 0.001 0.001"/>
     </geometry>
     <material name="silver"/>
@@ -20,5 +20,5 @@
     <origin xyz="0 0 0" rpy="0 0 0"/>
     <geometry>
-      <mesh filename="/home/cirp-lab/moore/prefab_robots/PingTi_Arm_v3/PingTi_Arm_5DOF_v4_copy_description/meshes/base_link.stl" scale="0.001 0.001 0.001"/>
+      <mesh filename="meshes/base_link.stl" scale="0.001 0.001 0.001"/>
     </geometry>
   </collision>
@@ -33,5 +33,5 @@
     <origin xyz="-0.04035 -0.73013 -0.397948" rpy="0 0 0"/>
     <geometry>
-      <mesh filename="/home/cirp-lab/moore/prefab_robots/PingTi_Arm_v3/PingTi_Arm_5DOF_v4_copy_description/meshes/elbow_link_1.stl" scale="0.001 0.001 0.001"/>
+      <mesh filename="meshes/elbow_link_1.stl" scale="0.001 0.001 0.001"/>
     </geometry>
     <material name="silver"/>
@@ -40,5 +40,5 @@
     <origin xyz="-0.04035 -0.73013 -0.397948" rpy="0 0 0"/>
     <geometry>
-      <mesh filename="/home/cirp-lab/moore/prefab_robots/PingTi_Arm_v3/PingTi_Arm_5DOF_v4_copy_description/meshes/elbow_link_1.stl" scale="0.001 0.001 0.001"/>
+      <mesh filename="meshes/elbow_link_1.stl" scale="0.001 0.001 0.001"/>
     </geometry>
   </collision>
@@ -53,5 +53,5 @@
     <origin xyz="-0.024329 -0.46443 -0.400273" rpy="0 0 0"/>
     <geometry>
-      <mesh filename="/home/cirp-lab/moore/prefab_robots/PingTi_Arm_v3/PingTi_Arm_5DOF_v4_copy_description/meshes/STS3215_wrist_pitch_1.stl" scale="0.001 0.001 0.001"/>
+      <mesh filename="meshes/STS3215_wrist_pitch_1.stl" scale="0.001 0.001 0.001"/>
     </geometry>
     <material name="silver"/>
@@ -60,5 +60,5 @@
     <origin xyz="-0.024329 -0.46443 -0.400273" rpy="0 0 0"/>
     <geometry>
-      <mesh filename="/home/cirp-lab/moore/prefab_robots/PingTi_Arm_v3/PingTi_Arm_5DOF_v4_copy_description/meshes/STS3215_wrist_pitch_1.stl" scale="0.001 0.001 0.001"/>
+      <mesh filename="meshes/STS3215_wrist_pitch_1.stl" scale="0.001 0.001 0.001"/>
     </geometry>
   </collision>
@@ -73,5 +73,5 @@
     <origin xyz="0.013571 -0.43998 -0.399823" rpy="0 0 0"/>
     <geometry>
-      <mesh filename="/home/cirp-lab/moore/prefab_robots/PingTi_Arm_v3/PingTi_Arm_5DOF_v4_copy_description/meshes/wrist_link_1.stl" scale="0.001 0.001 0.001"/>
+      <mesh filename="meshes/wrist_link_1.stl" scale="0.001 0.001 0.001"/>
     </geometry>
     <material name="silver"/>
@@ -80,5 +80,5 @@
     <origin xyz="0.013571 -0.43998 -0.399823" rpy="0 0 0"/>
     <geometry>
-      <mesh filename="/home/cirp-lab/moore/prefab_robots/PingTi_Arm_v3/PingTi_Arm_5DOF_v4_copy_description/meshes/wrist_link_1.stl" scale="0.001 0.001 0.001"/>
+      <mesh filename="meshes/wrist_link_1.stl" scale="0.001 0.001 0.001"/>
     </geometry>
   </collision>
@@ -93,5 +93,5 @@
     <origin xyz="-0.004529 -0.41776 -0.399823" rpy="0 0 0"/>
     <geometry>
-      <mesh filename="/home/cirp-lab/moore/prefab_robots/PingTi_Arm_v3/PingTi_Arm_5DOF_v4_copy_description/meshes/STS3215_wrist_roll_1.stl" scale="0.001 0.001 0.001"/>
+      <mesh filename="meshes/STS3215_wrist_roll_1.stl" scale="0.001 0.001 0.001"/>
     </geometry>
     <material name="silver"/>
@@ -100,5 +100,5 @@
     <origin xyz="-0.004529 -0.41776 -0.399823" rpy="0 0 0"/>
     <geometry>
-      <mesh filename="/home/cirp-lab/moore/prefab_robots/PingTi_Arm_v3/PingTi_Arm_5DOF_v4_copy_description/meshes/STS3215_wrist_roll_1.stl" scale="0.001 0.001 0.001"/>
+      <mesh filename="meshes/STS3215_wrist_roll_1.stl" scale="0.001 0.001 0.001"/>
     </geometry>
   </collision>
@@ -113,5 +113,5 @@
     <origin xyz="-0.006169 -0.37926 -0.400273" rpy="0 0 0"/>
     <geometry>
-      <mesh filename="/home/cirp-lab/moore/prefab_robots/PingTi_Arm_v3/PingTi_Arm_5DOF_v4_copy_description/meshes/gripper_mount_1.stl" scale="0.001 0.001 0.001"/>
+      <mesh filename="meshes/gripper_mount_1.stl" scale="0.001 0.001 0.001"/>
     </geometry>
     <material name="silver"/>
@@ -120,5 +120,5 @@
     <origin xyz="-0.006169 -0.37926 -0.400273" rpy="0 0 0"/>
     <geometry>
-      <mesh filename="/home/cirp-lab/moore/prefab_robots/PingTi_Arm_v3/PingTi_Arm_5DOF_v4_copy_description/meshes/gripper_mount_1.stl" scale="0.001 0.001 0.001"/>
+      <mesh filename="meshes/gripper_mount_1.stl" scale="0.001 0.001 0.001"/>
     </geometry>
   </collision>
@@ -133,5 +133,5 @@
     <origin xyz="0.010721 -0.36486 -0.402552" rpy="0 0 0"/>
     <geometry>
-      <mesh filename="/home/cirp-lab/moore/prefab_robots/PingTi_Arm_v3/PingTi_Arm_5DOF_v4_copy_description/meshes/STS3215_gripper_1.stl" scale="0.001 0.001 0.001"/>
+      <mesh filename="meshes/STS3215_gripper_1.stl" scale="0.001 0.001 0.001"/>
     </geometry>
     <material name="silver"/>
@@ -140,5 +140,5 @@
     <origin xyz="0.010721 -0.36486 -0.402552" rpy="0 0 0"/>
     <geometry>
-      <mesh filename="/home/cirp-lab/moore/prefab_robots/PingTi_Arm_v3/PingTi_Arm_5DOF_v4_copy_description/meshes/STS3215_gripper_1.stl" scale="0.001 0.001 0.001"/>
+      <mesh filename="meshes/STS3215_gripper_1.stl" scale="0.001 0.001 0.001"/>
     </geometry>
   </collision>
@@ -153,5 +153,5 @@
     <origin xyz="-0.024479 -0.36486 -0.382352" rpy="0 0 0"/>
     <geometry>
-      <mesh filename="/home/cirp-lab/moore/prefab_robots/PingTi_Arm_v3/PingTi_Arm_5DOF_v4_copy_description/meshes/moving_gripper_1.stl" scale="0.001 0.001 0.001"/>
+      <mesh filename="meshes/moving_gripper_1.stl" scale="0.001 0.001 0.001"/>
     </geometry>
     <material name="silver"/>
@@ -160,5 +160,5 @@
     <origin xyz="-0.024479 -0.36486 -0.382352" rpy="0 0 0"/>
     <geometry>
-      <mesh filename="/home/cirp-lab/moore/prefab_robots/PingTi_Arm_v3/PingTi_Arm_5DOF_v4_copy_description/meshes/moving_gripper_1.stl" scale="0.001 0.001 0.001"/>
+      <mesh filename="meshes/moving_gripper_1.stl" scale="0.001 0.001 0.001"/>
     </geometry>
   </collision>
@@ -173,5 +173,5 @@
     <origin xyz="0.017721 -0.47293 -0.399948" rpy="0 0 0"/>
     <geometry>
-      <mesh filename="/home/cirp-lab/moore/prefab_robots/PingTi_Arm_v3/PingTi_Arm_5DOF_v4_copy_description/meshes/wrist_mount_link_1.stl" scale="0.001 0.001 0.001"/>
+      <mesh filename="meshes/wrist_mount_link_1.stl" scale="0.001 0.001 0.001"/>
     </geometry>
     <material name="silver"/>
@@ -180,5 +180,5 @@
     <origin xyz="0.017721 -0.47293 -0.399948" rpy="0 0 0"/>
     <geometry>
-      <mesh filename="/home/cirp-lab/moore/prefab_robots/PingTi_Arm_v3/PingTi_Arm_5DOF_v4_copy_description/meshes/wrist_mount_link_1.stl" scale="0.001 0.001 0.001"/>
+      <mesh filename="meshes/wrist_mount_link_1.stl" scale="0.001 0.001 0.001"/>
     </geometry>
   </collision>
@@ -193,5 +193,5 @@
     <origin xyz="0.0 -0.78468 -0.092798" rpy="0 0 0"/>
     <geometry>
-      <mesh filename="/home/cirp-lab/moore/prefab_robots/PingTi_Arm_v3/PingTi_Arm_5DOF_v4_copy_description/meshes/STS3215_base_yaw_1.stl" scale="0.001 0.001 0.001"/>
+      <mesh filename="meshes/STS3215_base_yaw_1.stl" scale="0.001 0.001 0.001"/>
     </geometry>
     <material name="silver"/>
@@ -200,5 +200,5 @@
     <origin xyz="0.0 -0.78468 -0.092798" rpy="0 0 0"/>
     <geometry>
-      <mesh filename="/home/cirp-lab/moore/prefab_robots/PingTi_Arm_v3/PingTi_Arm_5DOF_v4_copy_description/meshes/STS3215_base_yaw_1.stl" scale="0.001 0.001 0.001"/>
+      <mesh filename="meshes/STS3215_base_yaw_1.stl" scale="0.001 0.001 0.001"/>
     </geometry>
   </collision>
@@ -213,5 +213,5 @@
     <origin xyz="0.0 -0.79488 -0.074498" rpy="0 0 0"/>
     <geometry>
-      <mesh filename="/home/cirp-lab/moore/prefab_robots/PingTi_Arm_v3/PingTi_Arm_5DOF_v4_copy_description/meshes/base_yaw_link_1.stl" scale="0.001 0.001 0.001"/>
+      <mesh filename="meshes/base_yaw_link_1.stl" scale="0.001 0.001 0.001"/>
     </geometry>
     <material name="silver"/>
@@ -220,5 +220,5 @@
     <origin xyz="0.0 -0.79488 -0.074498" rpy="0 0 0"/>
     <geometry>
-      <mesh filename="/home/cirp-lab/moore/prefab_robots/PingTi_Arm_v3/PingTi_Arm_5DOF_v4_copy_description/meshes/base_yaw_link_1.stl" scale="0.001 0.001 0.001"/>
+      <mesh filename="meshes/base_yaw_link_1.stl" scale="0.001 0.001 0.001"/>
     </geometry>
   </collision>
@@ -233,5 +233,5 @@
     <origin xyz="-0.020911 -0.76183 -0.131098" rpy="0 0 0"/>
     <geometry>
-      <mesh filename="/home/cirp-lab/moore/prefab_robots/PingTi_Arm_v3/PingTi_Arm_5DOF_v4_copy_description/meshes/STS3215_shoulder_pitch_1_1.stl" scale="0.001 0.001 0.001"/>
+      <mesh filename="meshes/STS3215_shoulder_pitch_1_1.stl" scale="0.001 0.001 0.001"/>
     </geometry>
     <material name="silver"/>
@@ -240,5 +240,5 @@
     <origin xyz="-0.020911 -0.76183 -0.131098" rpy="0 0 0"/>
     <geometry>
-      <mesh filename="/home/cirp-lab/moore/prefab_robots/PingTi_Arm_v3/PingTi_Arm_5DOF_v4_copy_description/meshes/STS3215_shoulder_pitch_1_1.stl" scale="0.001 0.001 0.001"/>
+      <mesh filename="meshes/STS3215_shoulder_pitch_1_1.stl" scale="0.001 0.001 0.001"/>
     </geometry>
   </collision>
@@ -253,5 +253,5 @@
     <origin xyz="0.020911 -0.76183 -0.131098" rpy="0 0 0"/>
     <geometry>
-      <mesh filename="/home/cirp-lab/moore/prefab_robots/PingTi_Arm_v3/PingTi_Arm_5DOF_v4_copy_description/meshes/STS3215_shoulder_pitch_2_1.stl" scale="0.001 0.001 0.001"/>
+      <mesh filename="meshes/STS3215_shoulder_pitch_2_1.stl" scale="0.001 0.001 0.001"/>
     </geometry>
     <material name="silver"/>
@@ -260,5 +260,5 @@
     <origin xyz="0.020911 -0.76183 -0.131098" rpy="0 0 0"/>
     <geometry>
-      <mesh filename="/home/cirp-lab/moore/prefab_robots/PingTi_Arm_v3/PingTi_Arm_5DOF_v4_copy_description/meshes/STS3215_shoulder_pitch_2_1.stl" scale="0.001 0.001 0.001"/>
+      <mesh filename="meshes/STS3215_shoulder_pitch_2_1.stl" scale="0.001 0.001 0.001"/>
     </geometry>
   </collision>
@@ -273,5 +273,5 @@
     <origin xyz="0.041111 -0.76183 -0.166298" rpy="0 0 0"/>
     <geometry>
-      <mesh filename="/home/cirp-lab/moore/prefab_robots/PingTi_Arm_v3/PingTi_Arm_5DOF_v4_copy_description/meshes/shoulder_link_1.stl" scale="0.001 0.001 0.001"/>
+      <mesh filename="meshes/shoulder_link_1.stl" scale="0.001 0.001 0.001"/>
     </geometry>
     <material name="silver"/>
@@ -280,5 +280,5 @@
     <origin xyz="0.041111 -0.76183 -0.166298" rpy="0 0 0"/>
     <geometry>
-      <mesh filename="/home/cirp-lab/moore/prefab_robots/PingTi_Arm_v3/PingTi_Arm_5DOF_v4_copy_description/meshes/shoulder_link_1.stl" scale="0.001 0.001 0.001"/>
+      <mesh filename="meshes/shoulder_link_1.stl" scale="0.001 0.001 0.001"/>
     </geometry>
   </collision>
@@ -293,5 +293,5 @@
     <origin xyz="0.020972 -0.76533 -0.397948" rpy="0 0 0"/>
     <geometry>
-      <mesh filename="/home/cirp-lab/moore/prefab_robots/PingTi_Arm_v3/PingTi_Arm_5DOF_v4_copy_description/meshes/STS3215_elbow_pitch_2_1.stl" scale="0.001 0.001 0.001"/>
+      <mesh filename="meshes/STS3215_elbow_pitch_2_1.stl" scale="0.001 0.001 0.001"/>
     </geometry>
     <material name="silver"/>
@@ -300,5 +300,5 @@
     <origin xyz="0.020972 -0.76533 -0.397948" rpy="0 0 0"/>
     <geometry>
-      <mesh filename="/home/cirp-lab/moore/prefab_robots/PingTi_Arm_v3/PingTi_Arm_5DOF_v4_copy_description/meshes/STS3215_elbow_pitch_2_1.stl" scale="0.001 0.001 0.001"/>
+      <mesh filename="meshes/STS3215_elbow_pitch_2_1.stl" scale="0.001 0.001 0.001"/>
     </geometry>
   </collision>
@@ -313,5 +313,5 @@
     <origin xyz="-0.02015 -0.76533 -0.397948" rpy="0 0 0"/>
     <geometry>
-      <mesh filename="/home/cirp-lab/moore/prefab_robots/PingTi_Arm_v3/PingTi_Arm_5DOF_v4_copy_description/meshes/STS3215_elbow_pitch_1_1.stl" scale="0.001 0.001 0.001"/>
+      <mesh filename="meshes/STS3215_elbow_pitch_1_1.stl" scale="0.001 0.001 0.001"/>
     </geometry>
     <material name="silver"/>
@@ -320,5 +320,5 @@
     <origin xyz="-0.02015 -0.76533 -0.397948" rpy="0 0 0"/>
     <geometry>
-      <mesh filename="/home/cirp-lab/moore/prefab_robots/PingTi_Arm_v3/PingTi_Arm_5DOF_v4_copy_description/meshes/STS3215_elbow_pitch_1_1.stl" scale="0.001 0.001 0.001"/>
+      <mesh filename="meshes/STS3215_elbow_pitch_1_1.stl" scale="0.001 0.001 0.001"/>
     </geometry>
   </collision>
