Commit message: updated the relative paths to the meshes in the urdf pingti file

File: src/isaac_so_arm101/robots/pingti/PingTi_Arm_5DOF_v4_copy.urdf (robot description, URDF)
Before this commit: robot pingti_arm, 7 links, 6 joints
Links:
- link base_link: geometry collision mesh filename=meshes/base_link.stl; collision mesh filename=meshes/sts3215_base_yaw.stl
- link base_yaw_link: geometry collision mesh filename=meshes/base_yaw_link.stl; collision mesh filename=meshes/sts3215_shoulder_pitch_1.stl
- link moving_gripper: geometry collision mesh filename=meshes/moving_gripper.stl; visual mesh filename=meshes/moving_gripper.stl
- link shoulder_link: geometry collision mesh filename=meshes/shoulder_link.stl; collision mesh filename=meshes/sts3215_elbow_pitch_1.stl
- link sts3215_gripper: geometry collision mesh filename=meshes/gripper_mount.stl; collision mesh filename=meshes/sts3215_gripper.stl
- link sts3215_wrist_roll: geometry collision mesh filename=meshes/sts3215_wrist_roll.stl; collision mesh filename=meshes/wrist_link.stl
- link wrist_mount_link: geometry collision mesh filename=meshes/elbow_link.stl; collision mesh filename=meshes/sts3215_wrist_pitch.stl

Commit message: updated the meshes folder with assests straight from onshape

File: src/isaac_so_arm101/robots/pingti/PingTi_Arm_5DOF_v4_copy.urdf (robot description, URDF)
Before this commit: robot pingti_arm, 7 links, 6 joints
Links:
- link base_link: geometry collision mesh filename=assets/base_link.stl; collision mesh filename=assets/sts3215_base_yaw.stl
- link base_yaw_link: geometry collision mesh filename=assets/base_yaw_link.stl; collision mesh filename=assets/sts3215_shoulder_pitch_1.stl
- link moving_gripper: geometry collision mesh filename=assets/moving_gripper.stl; visual mesh filename=assets/moving_gripper.stl
- link shoulder_link: geometry collision mesh filename=assets/shoulder_link.stl; collision mesh filename=assets/sts3215_elbow_pitch_1.stl
- link sts3215_gripper: geometry collision mesh filename=assets/gripper_mount.stl; collision mesh filename=assets/sts3215_gripper.stl
- link sts3215_wrist_roll: geometry collision mesh filename=assets/sts3215_wrist_roll.stl; collision mesh filename=assets/wrist_link.stl
- link wrist_mount_link: geometry collision mesh filename=assets/elbow_link.stl; collision mesh filename=assets/sts3215_wrist_pitch.stl
